Commit message: edit urdf - add laser sensors

File: pepper_description/urdf/pepper1.0_generated_urdf/pepperGazebo.xacro (robot description, xacro)
@@ -3,4 +3,5 @@
     <!-- MACROS FOR DISABLE LINKS -->
 	<xacro:property name="PI" value="3.14159265359" />
+    <xacro:property name="robot_namespace" value="/pepper_robot" />
     <xacro:macro name="DisabledLinks" params="side side_small">
         <plugin name="${side}Finger11_link" filename="libroboticsgroup_gazebo_disable_link_plugin.so">
@@ -692,7 +693,8 @@
 </gazebo>
 <!-- Drive controller -->
-<gazebo>
+<!---<gazebo>
   <plugin name="differential_drive_controller" filename="libgazebo_ros_diff_drive.so">
     <alwaysOn>true</alwaysOn>
+    <legacyMode>false</legacyMode>
     <updateRate>100</updateRate>
     <robotNamespace>/</robotNamespace>
@@ -705,6 +707,161 @@
     <odometryTopic>odom_diffdrive</odometryTopic>
     <odometryFrame>odom</odometryFrame>
-    <robotBaseFrame>base_footprint</robotBaseFrame>
+    <odometrySource>world</odometrySource>
+    <publishTf>1</publishTf>
+    <rosDebugLevel>na</rosDebugLevel>
+    <wheelAcceleration>0</wheelAcceleration>
+    <wheelTorque>5</wheelTorque>
+    <robotBaseFrame>base_link</robotBaseFrame>
+    <publishWheelTF>false</publishWheelTF>
+    <publishWheelJointState>false</publishWheelJointState>
   </plugin>
 </gazebo>
+-->
+    <gazebo>
+        <plugin name="base_drive_controller" filename="libpepper_gazebo_ros_force_omni_base.so">
+            <robotNamespace>${robot_namespace}</robotNamespace>
+            <commandTopic>cmd_vel</commandTopic>
+            <odometryTopic>odom</odometryTopic>
+            <publishOdometryTf>true</publishOdometryTf>
+            <odometryFrame>odom</odometryFrame>
+            <odometryRate>20.0</odometryRate>
+            <robotBaseFrame>Tibia</robotBaseFrame>
+            <yaw_velocity_p_gain>500.0</yaw_velocity_p_gain>
+            <yaw_velocity_i_gain>300.0</yaw_velocity_i_gain>
+            <x_velocity_p_gain>1000.0</x_velocity_p_gain>
+            <x_velocity_i_gain>300.0</x_velocity_i_gain>
+            <y_velocity_p_gain>1000.0</y_velocity_p_gain>
+            <y_velocity_i_gain>300.0</y_velocity_i_gain>
+            <max_torque>8.0</max_torque>
+            <max_force>3000.0</max_force>
+        </plugin>
+    </gazebo>
+    <!-- Lasers sensors -->
+    <!-- These are like pepper has in his hardware, however
+         the official naoqi ROS driver makes the merge of all the laser and references them to base_footprint frame
+    -->
+    <gazebo reference="SurroundingRightLaser_frame">
+      <sensor type="ray" name="laser_sensor_right">
+        <pose>0 0 0 0 0 0</pose>
+        <visualize>true</visualize>
+        <update_rate>10</update_rate>
+        <ray>
+          <scan>
+            <horizontal>
+              <samples>15</samples>
+              <resolution>1</resolution>
+              <min_angle>-0.515</min_angle>
+              <max_angle>0.515</max_angle>
+            </horizontal>
+          </scan>
+          <range>
+            <min>0.10</min>
+            <max>6.5</max>
+            <resolution>0.01</resolution>
+          </range>
+          <noise>
+            <type>gaussian</type>
+            <mean>0.0</mean>
+            <stddev>0.01</stddev>
+          </noise>
+        </ray>
+        <plugin name="gazebo_ros_laser_sensor_right_plugin" filename="libgazebo_ros_laser.so">
+          <topicName>${robot_namespace}/laser/right</topicName>
+          <frameName>SurroundingRightLaser_frame</frameName>
+        </plugin>
+      </sensor>
+    </gazebo>
+    <gazebo reference="SurroundingLeftLaser_frame">
+      <sensor type="ray" name="laser_sensor_left">
+        <pose>0 0 0 0 0 0</pose>
+        <visualize>true</visualize>
+        <update_rate>10</update_rate>
+        <ray>
+          <scan>
+            <horizontal>
+              <samples>15</samples>
+              <resolution>1</resolution>
+              <min_angle>-0.515</min_angle>
+              <max_angle>0.515</max_angle>
+            </horizontal>
+          </scan>
+          <range>
+            <min>0.10</min>
+            <max>6.5</max>
+            <resolution>0.01</resolution>
+          </range>
+          <noise>
+            <type>gaussian</type>
+            <mean>0.0</mean>
+            <stddev>0.01</stddev>
+          </noise>
+        </ray>
+        <plugin name="gazebo_ros_laser_sensor_left_plugin" filename="libgazebo_ros_laser.so">
+          <topicName>${robot_namespace}/laser/left</topicName>
+          <frameName>SurroundingLeftLaser_frame</frameName>
+        </plugin>
+      </sensor>
+    </gazebo>
+    <gazebo reference="SurroundingFrontLaser_frame">
+      <sensor type="ray" name="laser_sensor_front">
+        <pose>0 0 0 0 0 0</pose>
+        <visualize>true</visualize>
+        <update_rate>10</update_rate>
+        <ray>
+          <scan>
+            <horizontal>
+              <samples>15</samples>
+              <resolution>1</resolution>
+              <min_angle>-0.515</min_angle>
+              <max_angle>0.515</max_angle>
+            </horizontal>
+          </scan>
+          <range>
+            <min>0.10</min>
+            <max>6.5</max>
+            <resolution>0.01</resolution>
+          </range>
+          <noise>
+            <type>gaussian</type>
+            <mean>0.0</mean>
+            <stddev>0.01</stddev>
+          </noise>
+        </ray>
+        <plugin name="gazebo_ros_laser_sensor_front_plugin" filename="libgazebo_ros_laser.so">
+          <topicName>${robot_namespace}/laser/front</topicName>
+          <frameName>SurroundingFrontLaser_frame</frameName>
+        </plugin>
+      </sensor>
+    </gazebo> -->
+    <!--gazebo reference="base_footprint">
+      <sensor type="ray" name="laser">
+        <pose>0 0 0 0 0 0</pose>
+        <visualize>false</visualize>
+        <update_rate>10</update_rate>
+        <ray>
+          <scan>
+            <horizontal>
+              <samples>45</samples>
+              <resolution>1</resolution>
+              <min_angle>-2.09439992905</min_angle>
+              <max_angle>2.09439992905</max_angle>
+            </horizontal>
+          </scan>
+          <range>
+            <min>0.10</min>
+            <max>6.5</max>
+            <resolution>0.01</resolution>
+          </range>
+          <noise>
+            <type>gaussian</type>
+            <mean>0.0</mean>
+            <stddev>0.01</stddev>
+          </noise>
+        </ray>
+        <plugin name="gazebo_ros_laser_sensor_front_plugin" filename="libgazebo_ros_laser.so">
+          <topicName>${robot_namespace}/laser</topicName>
+          <frameName>base_footprint</frameName>
+        </plugin>
+      </sensor>
+    </gazebo-->
 </robot>

File: pepper_description/urdf/pepper1.0_generated_urdf/pepper_visual_collisions.xacro (robot description, xacro)
@@ -111,5 +111,6 @@
 		<collision>
 			<geometry>
-				<mesh filename="package://pepper_meshes/meshes/1.0/WheelFL_0.10.stl" scale="0.1 0.1 0.1"/>
+				<!--mesh filename="package://pepper_meshes/meshes/1.0/WheelFL_0.10.stl" scale="0.1 0.1 0.1"/-->
+                                <sphere radius="0.09"/>
 			</geometry>
 			<origin rpy="0 0 0" xyz="0 0 0"/>
@@ -251,5 +252,6 @@
 		<collision>
 			<geometry>
-				<mesh filename="package://pepper_meshes/meshes/1.0/KneePitch_0.10.stl" scale="0.1 0.1 0.1"/>
+				<cylinder length="0.05" radius="0.1"/>
+				<!--mesh filename="package://pepper_meshes/meshes/1.0/KneePitch_0.10.stl" scale="0.1 0.1 0.1"/-->
 			</geometry>
 			<origin rpy="0 0 0" xyz="0 0 0"/>
@@ -461,5 +463,6 @@
 		<collision>
 			<geometry>
-				<mesh filename="package://pepper_meshes/meshes/1.0/WheelB_0.10.stl" scale="0.1 0.1 0.1"/>
+				<!--mesh filename="package://pepper_meshes/meshes/1.0/WheelB_0.10.stl" scale="0.1 0.1 0.1"/-->  <!-- wheels of radius 0.14 meter-->
+				<sphere radius="0.09"/>
 			</geometry>
 			<origin rpy="0 0 0" xyz="0 0 0"/>
@@ -629,5 +632,6 @@
 		<collision>
 			<geometry>
-				<mesh filename="package://pepper_meshes/meshes/1.0/WheelFR_0.10.stl" scale="0.1 0.1 0.1"/>
+				<!--mesh filename="package://pepper_meshes/meshes/1.0/WheelFR_0.10.stl" scale="0.1 0.1 0.1"/-->
+				<sphere radius="0.09"/>
 			</geometry>
 			<origin rpy="0 0 0" xyz="0 0 0"/>
